File: pcb/project/portcullis/portcullis.kicad_sch (KiCad schematic)
At the start: 0 parts

Commit message: pcb
Parts:
- added A1: Arduino_UNO_R3, Arduino_UNOR3:ARDUINO_ARDUINO_UNO_REV3, symbol MCU_Module:Arduino_UNO_R3
- added M1: Motor_Servo_Pos (Rotational), symbol Motor:Motor_Servo
- added M2: Motor_Servo_Cont (Linear), symbol Motor:Motor_Servo
- added U1: i2c_LCD, i2c_LCD:i2c_LCD, symbol i2c_LCD:i2c_LCD
- added U2: ~, symbol 4x4_keypad:4x4_keypad
Connections:
- new net: A1.26 (D11), M2.1 (PWM)
- new net: A1.25 (D10), M1.1 (PWM)
- new net: A1.17 (D2), U2.1 (C1)
- new net: A1.18 (D3), U2.2 (C2)
- new net: A1.19 (D4), U2.3 (C3)
- new net: A1.20 (D5), U2.4 (C4)
- new net: A1.21 (D6), U2.5 (R1)
- new net: A1.22 (D7), U2.6 (R2)
- new net: A1.23 (D8), U2.7 (R3)
- new net: A1.24 (D9), U2.8 (R4)
- new net: A1.13 (SDA/A4), U1.3 (SDA)
- new net: A1.14 (SCL/A5), U1.4 (SCL)
- new net +5V: A1.5 (+5V), M1.2 (+), M2.2 (+), U1.2 (VCC)
- new net GND: A1.29 (GND), M1.3 (-), M2.3 (-), U1.1 (GND)

Commit message: pcb finish pt 1
Parts:
- M1, M2: footprint (none) -> Servo:3-Pin Servo
- U2: footprint (none) -> Keypad:4x4 16 Button Keypad
Changed lines of the file:
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@@
 			)
 		)
-		(property "Footprint" ""
+		(property "Footprint" "Servo:3-Pin Servo"
 			(at 154.686 60.96 0)
 			(effects
@@
 			)
 		)
-		(property "Footprint" ""
+		(property "Footprint" "Servo:3-Pin Servo"
 			(at 97.536 60.96 0)
 			(effects
@@
 			)
 		)
-		(property "Footprint" ""
+		(property "Footprint" "Keypad:4x4 16 Button Keypad"
 			(at 119.38 38.1 0)
 			(effects

Commit message: final
Parts:
- added R1: 330Ω, symbol Device:R
- added U3: ~, symbol 19mmMomentaryPushbutton:19mmMomentaryPushbutton
Connections:
- net GND: now also U3. (LED_GND)
- net at A1.27 (D12): now also R1.2
- net at A1.28 (D13): now also U3. (LED_GND)
- new net: R1.1, U3. (LED_GND)
